File: eagle/patch-panel/patch-panel.sch (EAGLE design)
At the start: 61 parts, among them IC1 LM741D, IC10 LM741D, IC2 LM741D, IC3 LM741D, IC4 LM741D, IC5 LM741D, IC6 LM741D, IC7 LM741D, IC8 LM741D, IC9 LM741D, X1 1751251, X10 1751248, X11 1751248, X2 1751248, X3 1751248, X4 1751248, X5 1751248, X6 1751248, X7 1751248, X8 1751248, X9 1751248

Commit message: Fix patch panel design to use correct pot pin
Parts:
- removed IC10, IC4, IC5, IC6, IC7, IC8, IC9: LM741D, linear:LM741D
- removed R13, R14, R15, R17, R18, R19, R21, R22, R23, R25, R26, R27, R29, R30, R31, R33, R34, R35, R37, R38, R39: 10K, rcl:R-EU_M1206
- removed R16, R20, R24, R28, R32, R36, R40: 10K, bourns-PTVA09A-4:PTVA09A-4
- removed X10, X11, X2, X3, X4, X5, X6, X7, X8, X9: 1751248, con-phoenix-350:1751248
- added PAD1, PAD2, PAD3, PAD4, PAD5, PAD6: (no value), wirepad:2,54/1,0
Connections:
- removed net GND: R1.1, R12.WIPER, R13.1, R16.WIPER, R17.1, R20.WIPER, R21.1, R24.WIPER, R25.1, R28.WIPER, R29.1, R32.WIPER, R33.1, R36.WIPER, R37.1, R4.WIPER, R40.WIPER, R5.1, R8.WIPER, R9.1, X1-2.K
- removed net N$12: R7.1, X3-1.K
- removed net N$14 (its old number): IC3.OUT, R10.1, X4-2.K
- removed net N$18: R11.1, X4-1.K
- removed net N$19: IC4.-IN, R13.2, R14.2
- removed net N$20: IC4.OUT, R14.1, X5-2.K
- removed net N$21: IC4.+IN, R15.2, R16.B
- removed net N$24: R15.1, X5-1.K
- removed net N$25: IC5.-IN, R17.2, R18.2
- removed net N$26: IC5.OUT, R18.1, X6-2.K
- removed net N$27: IC5.+IN, R19.2, R20.B
- removed net N$30: R19.1, X6-1.K
- removed net N$31: IC6.-IN, R21.2, R22.2
- removed net N$32: IC6.OUT, R22.1, X7-2.K
- removed net N$33: IC6.+IN, R23.2, R24.B
- removed net N$36: R23.1, X7-1.K
- removed net N$37: IC7.-IN, R25.2, R26.2
- removed net N$38: IC7.OUT, R26.1, X8-2.K
- removed net N$39: IC7.+IN, R27.2, R28.B
- removed net N$42: R27.1, X8-1.K
- removed net N$43: IC8.-IN, R29.2, R30.2
- removed net N$44: IC8.OUT, R30.1, X9-2.K
- removed net N$45: IC8.+IN, R31.2, R32.B
- removed net N$48: R31.1, X9-1.K
- removed net N$49: IC9.-IN, R33.2, R34.2
- removed net N$50: IC9.OUT, R34.1, X10-2.K
- removed net N$51: IC9.+IN, R35.2, R36.B
- removed net N$54: R35.1, X10-1.K
- removed net N$55: IC10.-IN, R37.2, R38.2
- removed net N$56: IC10.OUT, R38.1, X11-2.K
- removed net N$57: IC10.+IN, R39.2, R40.B
- removed net N$60: R39.1, X11-1.K
- new net N$10: PAD3.P, R7.1
- new net N$16: IC3.+IN, R11.2, R12.A
- new net N$17: PAD5.P, R11.1
- new net N$40: IC1.V-, IC2.V-, IC3.V-, X1-3.K
- net N$11: now also IC1.V+, IC2.V+, IC3.V+, X1-1.K; no longer IC1.V-, IC10.V-, IC2.V-, IC3.V-, IC4.V-, IC5.V-, IC6.V-, IC7.V-, IC8.V-, IC9.V-, X1-3.K
- net N$15: now also IC3.OUT, PAD6.P, R10.1; no longer IC3.+IN, R11.2, R12.B
- net N$2: now also PAD2.P; no longer X2-2.K
- net N$3: now also R4.A; no longer R4.B
- net N$5: now also R1.1, R12.WIPER, R4.WIPER, R5.1, R8.WIPER, R9.1, X1-2.K; no longer IC1.V+, IC10.V+, IC2.V+, IC3.V+, IC4.V+, IC5.V+, IC6.V+, IC7.V+, IC8.V+, IC9.V+, X1-1.K
- net N$6: now also PAD1.P; no longer X2-1.K
- net N$8: now also PAD4.P; no longer X3-2.K
- net N$9: now also R8.A; no longer R8.B
Other:
- note removed: "Output"
- moved on the sheet: R12, R4, R8
