File: modules/midi-in/eagle/cv-board/cv-board.sch (EAGLE design)
At the start: 50 parts, among them IC2 TL072P, IC3 TL074P, IC4 TL074P, T1 BC547, T2 BC547, X1 POWER IN

Commit message: Finish CV board,
Connections:
- net VCC renamed N$30
Changed lines of the file:
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@@
 </segment>
 </net>
-<net name="N$31" class="0">
+<net name="N$3" class="0">
 <segment>
 <pinref part="R20" gate="G$1" pin="2"/>
@@
 </segment>
 </net>
-<net name="VCC" class="0">
+<net name="N$30" class="0">
 <segment>
 <pinref part="T2" gate="G$1" pin="C"/>
