File: modules/distortion/kicad/distortion.kicad_pcb (KiCad board)
At the start: 2 copper layers, 50 x 132.2 mm, 60 parts, among them P1 CONN_01X03, P10 CONN_01X03, P11 CONN_01X03, P12 CONN_01X03, P13 CONN_01X03, P14 CONN_01X03, P2 CONN_01X03, P3 CONN_01X03, P4 CONN_01X03, P5 CONN_01X03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

Commit message: Final tweaks to distortion pcb
Parts:
- moved C7 27.3 mm to (105.4, 147.1)
- moved R17 27.3 mm to (104.6, 80.8)
- moved R18 27.3 mm to (104.6, 61.2)
- moved R3 27.3 mm to (104.6, 55.6)
- moved U3 27.3 mm to (105.4, 127.5)
- moved C10 27.3 mm to (90.9, 165.6)
- moved C2 27.3 mm to (96.3, 155.4)
- moved C4 27.3 mm to (109.0, 113.0)
- moved C5 27.3 mm to (84.3, 133.9)
- moved C6 27.3 mm to (78.2, 133.9)
- moved C8 27.3 mm to (99.3, 147.1)
- moved C9 27.3 mm to (84.3, 157.7)
- moved P1 27.3 mm to (66.8, 164.1)
- moved P10 27.3 mm to (66.0, 135.4)
- moved P12 27.3 mm to (110.2, 74.2)
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Other:
- outline, holes or cut-outs redrawn
- board text added: "BOARD 1 OF 2"
- board text added: "BOARD 2 OF 2"
- board text added: "POST-GAIN"
- board text added: "PRE-GAIN"
- board text removed: "BOARD 1/2"
- board text removed: "BOARD 2/2"
- board text removed: "POST GAIN"
- board text removed: "PRE GAIN"
