File: modules/clock-generator/kicad/clock-generator.sch (KiCad schematic (older format))
At the start: 22 parts, among them IC1 ATTINY84-S, P1 CONN_01X03, P2 CONN_02X03, P3 CONN_01X09, Q1 Q_NPN_BEC, SW1 SW_PUSH, SW2 SW_PUSH, U1 MAX7221, U2 4024, Y1 16MHz

Commit message: Finish clock generator PCB, start panel
Parts:
- P2: footprint Pin_Headers:Pin_Header_Angled_2x03_Pitch2.54mm -> Pin_Headers:Pin_Header_Straight_2x03_Pitch2.54mm
Connections:
- no-connect marks 9 -> 8
Other:
- moved on the sheet: C1, C2, C3, C4, P1
Changed lines of the file:
@@
 F 0 "P2" H 2650 4350 50  0000 C CNN
 F 1 "CONN_02X03" H 2650 3950 50  0000 C CNN
-F 2 "Pin_Headers:Pin_Header_Angled_2x03_Pitch2.54mm" H 2650 2950 50  0001 C CNN
+F 2 "Pin_Headers:Pin_Header_Straight_2x03_Pitch2.54mm" H 2650 2950 50  0001 C CNN
 F 3 "" H 2650 2950 50  0000 C CNN
 	1    2650 4150
@@
 L C C4
 U 1 1 5A10416F
-P 2600 5550
-F 0 "C4" H 2625 5650 50  0000 L CNN
-F 1 "100n" H 2625 5450 50  0000 L CNN
-F 2 "Capacitors_SMD:C_0805" H 2638 5400 50  0001 C CNN
-F 3 "" H 2600 5550 50  0000 C CNN
-	1    2600 5550
+P 2650 5050
+F 0 "C4" H 2675 5150 50  0000 L CNN
+F 1 "100n" H 2675 4950 50  0000 L CNN
+F 2 "Capacitors_SMD:C_0805" H 2688 4900 50  0001 C CNN
+F 3 "" H 2650 5050 50  0000 C CNN
+	1    2650 5050
 	1    0    0    -1
 $EndComp
@@
 L CP C2
 U 1 1 5A1044F4
-P 2100 5550
-F 0 "C2" H 2125 5650 50  0000 L CNN
-F 1 "10u" H 2125 5450 50  0000 L CNN
-F 2 "Capacitors_SMD:C_1206" H 2138 5400 50  0001 C CNN
-F 3 "" H 2100 5550 50  0000 C CNN
-	1    2100 5550
+P 2150 5050
+F 0 "C2" H 2175 5150 50  0000 L CNN
+F 1 "10u" H 2175 4950 50  0000 L CNN
+F 2 "Capacitors_SMD:C_1206" H 2188 4900 50  0001 C CNN
+F 3 "" H 2150 5050 50  0000 C CNN
+	1    2150 5050
 	1    0    0    -1
 $EndComp
@@
 L C C3
 U 1 1 5A105034
-P 2350 5550
-F 0 "C3" H 2375 5650 50  0000 L CNN
-F 1 "100n" H 2375 5450 50  0000 L CNN
-F 2 "Capacitors_SMD:C_0805" H 2388 5400 50  0001 C CNN
-F 3 "" H 2350 5550 50  0000 C CNN
-	1    2350 5550
+P 2400 5050
+F 0 "C3" H 2425 5150 50  0000 L CNN
+F 1 "100n" H 2425 4950 50  0000 L CNN
+F 2 "Capacitors_SMD:C_0805" H 2438 4900 50  0001 C CNN
+F 3 "" H 2400 5050 50  0000 C CNN
+	1    2400 5050
 	1    0    0    -1
 $EndComp
@@
 L CONN_01X03 P1
 U 1 1 5A106635
-P 1350 5600
-F 0 "P1" H 1350 5800 50  0000 C CNN
-F 1 "CONN_01X03" V 1450 5600 50  0000 C CNN
-F 2 "Connectors_Molex:Molex_KK-6410-03_03x2.54mm_Straight" H 1350 5600 50  0001 C CNN
-F 3 "" H 1350 5600 50  0000 C CNN
-	1    1350 5600
+P 1400 5100
+F 0 "P1" H 1400 5300 50  0000 C CNN
+F 1 "CONN_01X03" V 1500 5100 50  0000 C CNN
+F 2 "Connectors_Molex:Molex_KK-6410-03_03x2.54mm_Straight" H 1400 5100 50  0001 C CNN
+F 3 "" H 1400 5100 50  0000 C CNN
+	1    1400 5100
 	-1   0    0    1
 $EndComp
@@
 L CP C1
 U 1 1 5A109572
-P 1800 5550
-F 0 "C1" H 1825 5650 50  0000 L CNN
-F 1 "100u" H 1825 5450 50  0000 L CNN
-F 2 "Capacitors_ThroughHole:CP_Radial_D5.0mm_P2.00mm" H 1838 5400 50  0001 C CNN
-F 3 "" H 1800 5550 50  0000 C CNN
-	1    1800 5550
+P 1850 5050
+F 0 "C1" H 1875 5150 50  0000 L CNN
+F 1 "100u" H 1875 4950 50  0000 L CNN
+F 2 "Capacitors_ThroughHole:CP_Radial_D5.0mm_P2.00mm" H 1888 4900 50  0001 C CNN
+F 3 "" H 1850 5050 50  0000 C CNN
+	1    1850 5050
 	1    0    0    -1
 $EndComp
@@
 L PWR_FLAG #FLG01
 U 1 1 5A109713
-P 1550 5250
-F 0 "#FLG01" H 1550 5345 50  0001 C CNN
-F 1 "PWR_FLAG" H 1550 5430 50  0000 C CNN
-F 2 "" H 1550 5250 50  0000 C CNN
-F 3 "" H 1550 5250 50  0000 C CNN
-	1    1550 5250
+P 1600 4750
+F 0 "#FLG01" H 1600 4845 50  0001 C CNN
+F 1 "PWR_FLAG" H 1600 4930 50  0000 C CNN
+F 2 "" H 1600 4750 50  0000 C CNN
+F 3 "" H 1600 4750 50  0000 C CNN
+	1    1600 4750
 	0    -1   -1   0
 $EndComp
@@
 L VCC #PWR02
 U 1 1 5A109E76
-P 1600 5200
-F 0 "#PWR02" H 1600 5050 50  0001 C CNN
-F 1 "VCC" H 1600 5350 50  0000 C CNN
-F 2 "" H 1600 5200 50  0000 C CNN
-F 3 "" H 1600 5200 50  0000 C CNN
-	1    1600 5200
+P 1650 4700
+F 0 "#PWR02" H 1650 4550 50  0001 C CNN
+F 1 "VCC" H 1650 4850 50  0000 C CNN
+F 2 "" H 1650 4700 50  0000 C CNN
+F 3 "" H 1650 4700 50  0000 C CNN
+	1    1650 4700
 	1    0    0    -1
 $EndComp
@@
 L GND #PWR03
 U 1 1 5A10A57E
-P 1600 6100
-F 0 "#PWR03" H 1600 5850 50  0001 C CNN
-F 1 "GND" H 1600 5950 50  0000 C CNN
-F 2 "" H 1600 6100 50  0000 C CNN
-F 3 "" H 1600 6100 50  0000 C CNN
-	1    1600 6100
+P 1650 5600
+F 0 "#PWR03" H 1650 5350 50  0001 C CNN
+F 1 "GND" H 1650 5450 50  0000 C CNN
+F 2 "" H 1650 5600 50  0000 C CNN
+F 3 "" H 1650 5600 50  0000 C CNN
+	1    1650 5600
 	1    0    0    -1
 $EndComp
@@
 L PWR_FLAG #FLG04
 U 1 1 5A10A5B0
-P 1500 6050
-F 0 "#FLG04" H 1500 6145 50  0001 C CNN
-F 1 "PWR_FLAG" H 1500 6230 50  0000 C CNN
-F 2 "" H 1500 6050 50  0000 C CNN
-F 3 "" H 1500 6050 50  0000 C CNN
-	1    1500 6050
+P 1550 5550
+F 0 "#FLG04" H 1550 5645 50  0001 C CNN
+F 1 "PWR_FLAG" H 1550 5730 50  0000 C CNN
+F 2 "" H 1550 5550 50  0000 C CNN
+F 3 "" H 1550 5550 50  0000 C CNN
+	1    1550 5550
 	0    -1   -1   0
 $EndComp
-NoConn ~ 1550 5700
+NoConn ~ 1600 5200
 $Comp
 L GND #PWR05
@@
 NoConn ~ 6300 3300
 Wire Wire Line
-	1600 5500 1550 5500
-Wire Wire Line
-	1600 5200 1600 5500
-Wire Wire Line
-	1600 5250 1550 5250
-Connection ~ 1600 5250
-Wire Wire Line
-	1550 5600 1600 5600
-Wire Wire Line
-	1600 5600 1600 6100
-Wire Wire Line
-	1500 6050 1600 6050
-Connection ~ 1600 6050
-Wire Wire Line
-	1800 5400 1800 5350
-Connection ~ 1600 5350
-Wire Wire Line
-	1800 5700 1800 5750
-Connection ~ 1600 5750
+	1650 5000 1600 5000
+Wire Wire Line
+	1650 4700 1650 5000
+Wire Wire Line
+	1650 4750 1600 4750
+Connection ~ 1650 4750
+Wire Wire Line
+	1600 5100 1650 5100
+Wire Wire Line
+	1650 5100 1650 5600
+Wire Wire Line
+	1550 5550 1650 5550
+Connection ~ 1650 5550
+Wire Wire Line
+	1850 4900 1850 4850
+Connection ~ 1650 4850
+Wire Wire Line
+	1850 5200 1850 5250
+Connection ~ 1650 5250
 Wire Wire Line
 	3850 3000 3850 2950
@@
 Connection ~ 4300 3350
 Wire Wire Line
-	2100 5350 2100 5400
-Connection ~ 1800 5350
-Wire Wire Line
-	2350 5350 2350 5400
-Connection ~ 2100 5350
-Wire Wire Line
-	2600 5350 2600 5400
-Connection ~ 2350 5350
-Wire Wire Line
-	2100 5750 2100 5700
-Connection ~ 1800 5750
-Wire Wire Line
-	2350 5750 2350 5700
-Connection ~ 2100 5750
-Wire Wire Line
-	2600 5750 2600 5700
-Connection ~ 2350 5750
+	2150 4850 2150 4900
+Connection ~ 1850 4850
+Wire Wire Line
+	2400 4850 2400 4900
+Connection ~ 2150 4850
+Wire Wire Line
+	2650 4850 2650 4900
+Connection ~ 2400 4850
+Wire Wire Line
+	2150 5250 2150 5200
+Connection ~ 1850 5250
+Wire Wire Line
+	2400 5250 2400 5200
+Connection ~ 2150 5250
+Wire Wire Line
+	2650 5250 2650 5200
+Connection ~ 2400 5250
 Wire Wire Line
 	1000 2150 1000 2200
@@
 Text Notes 9250 4350 0    60   ~ 0
 BPM indicator LED
-Text Notes 1850 6000 0    60   ~ 0
+Text Notes 1900 5500 0    60   ~ 0
 Decoupling caps
 Text Notes 2350 4250 2    60   ~ 0
 ISP\nconnector
 NoConn ~ 3150 3300
-NoConn ~ 3300 1750
-Wire Wire Line
-	1600 5350 2600 5350
-Wire Wire Line
-	2600 5750 1600 5750
+Wire Wire Line
+	1650 4850 2650 4850
+Wire Wire Line
+	2650 5250 1650 5250
 $EndSCHEMATC
