File: modules/sequencer/kicad/sequencer.sch (KiCad schematic (older format))
At the start: 8 parts

Commit message: [WiP] Sequencer schematic
Parts:
- removed AFF?: CC56-12, symbol CC56-12
- removed U? (x2): 4051, symbol 4051
- removed U? (x2): TL072, symbol TL072
- added AFF?: CC04-41SURKWA, symbol CC04-41SURKWA
- added C?: 330n, symbol C
- added C?: 1u, symbol C
- added D? (x3): LED, symbol LED
- added Q? (x9): MMBT3906, SOT-23, symbol MMBT3906
- added R?: 22k, symbol R
- added R? (x10): 1k, symbol R
- added R? (x13): 10k, symbol R
- added R?: 330R, symbol R
- added R?: 220k, symbol R
- added R? (x2): 100k, symbol R
- added R?: 20k, symbol R
- added R?: 2k2, symbol R
- added RV? (x8): 100k, symbol LED-POT
- added RV? (x9): 100k, symbol POT
- added RV?: 1k, symbol POT
- added RV?: 3k3, symbol POT
- added SW? (x8): SW_PUSH_DPDT, symbol SW_PUSH_DPDT
- added SW? (x10): SW_PUSH_SMALL_H, symbol SW_PUSH_SMALL_H
- added SW?: SWITCH_INV_MSM, symbol SWITCH_INV_MSM
- added SW?: Switch_SPDT_x2, symbol Switch_SPDT_x2
- added U?: MCP3202, symbol MCP3202
- added U? (x2): CD4051, symbol CD4051
- added U?: ATmega32U4-AU, symbol ATmega32U4-AU
- added U?: MCP23S17, symbol MCP23S17
- added U? (x4): TL074, symbol TL074
- added U?: DG417, symbol DG417
Connections:
- net GND: now also U?.4 (E1), U?.4 (GND), U?.5 (E2), U?.5 (~LDAC~), U?.7 (AVSS), U?.9 (GND), C?.2, C?.2, R?.1, R?.1, R?.2, R?.2, RV?.1, RV?.1, RV?.1, RV?.1, RV?.1, RV?.1, RV?.1, RV?.1, SW?.2, SW?.2, SW?.2, SW?.2, SW?.2, SW?.2, SW?.2, SW?.2, SW?.2, SW?.2, SW?.2, U?.10 (VSS), U?.15 (A0), U?.16 (A1), U?.17 (A2), U?.3 (GND), U?.4 (Vss), U?.5 (+), U?.6 (INH), U?.6 (INH), U?.7 (VEE), U?.8 (VSS), U?.8 (VSS)
- net VCC: now also U?.1 (VDD), U?.19 (V+), U?.6 (VrefA), Q?.2 (E), R?.1, R?.1, R?.1, RV?.1, RV?.1, RV?.1, RV?.1, RV?.1, RV?.1, RV?.1, RV?.1, RV?.3, RV?.3, RV?.3, RV?.3, RV?.3, RV?.3, RV?.3, RV?.3, RV?.B, RV?.B, RV?.B, RV?.B, RV?.B, RV?.B, RV?.B, RV?.B, SW?.1, SW?.6, U?.16 (VDD), U?.16 (VDD), U?.18 (RESET), U?.4 (V+), U?.4 (V+), U?.5 (VCC), U?.8 (Vdd), U?.9 (VDD)
- net SPI_MOSI: now reaches U?.1 (DIN)
- net SPI_MOSI: now also U?.4 (SDI), U?.13 (SI), U?.5 (DIN)
- net at U?.11 (DIG_1): now also AFF?.5 (Dig2)
- net SPI_CS_DISPLAY: now reaches U?.12 (CS)
- net SPI_SCK: now reaches U?.13 (CLK)
- net SPI_SCK: now also U?.3 (SCK), U?.12 (SCK), U?.7 (CLK)
- net at U?.14 (SEG_A): now also AFF?.12 (a3,4), AFF?.17 (a1,2), D?.2 (A)
- net at U?.15 (SEG_F): now also AFF?.13 (f3,4), AFF?.18 (f1,2)
- net at U?.16 (SEG_B): now also AFF?.11 (b3,4), AFF?.16 (b1,2), D?.2 (A)
- net at U?.17 (SEG_G): now also AFF?.14 (g3,4), AFF?.19 (g1,2)
- net at U?.18 (ISET): now also R?.2
- net at U?.2 (DIG_0): now also AFF?.20 (Dig1)
- net at U?.20 (SEG_C): now also AFF?.4 (c1,2), AFF?.9 (c3,4), D?.2 (A)
- net at U?.21 (SEG_E): now also AFF?.3 (e1,2), AFF?.8 (e3,4)
- net at U?.22 (SEG_DP): now also AFF?.2 (DP1,2), AFF?.7 (DP3,4)
- net at U?.23 (SEG_D): now also AFF?.1 (d1,2), AFF?.6 (d3,4)
- net at U?.3 (DIG_4): now also D?.1 (K), D?.1 (K), D?.1 (K)
- net at U?.6 (DIG_2): now also AFF?.15 (Dig3)
- net at U?.7 (DIG_3): now also AFF?.10 (dig4)
- net STEP_A0: now reaches U?.1 (A0)
- net STEP_A0: now also U?.11 (A), U?.11 (A)
- net at U?.10 (O5): now also R?.1
- net at U?.11 (O4): now also R?.1
- net at U?.12 (O3): now also R?.1
- net at U?.13 (O2): now also R?.1
- net at U?.14 (O1): now also R?.1
- net at U?.15 (O0): now also R?.1
- net STEP_A1: now reaches U?.2 (A1)
- net STEP_A1: now also U?.10 (B), U?.10 (B)
- net STEP_A2: now reaches U?.3 (A2)
- net STEP_A2: now also U?.9 (C), U?.9 (C)
- net DECODER_ENABLE: now reaches U?.6 (E3)
- net at U?.7 (O7): now also R?.1
- net at U?.9 (O6): now also R?.1
- net SPI_CS_DAC: now reaches U?.2 (~CS~)
- net at U?.8 (VoutA): now also R?.2
- new net: U?.2 (CH0), U?.3 (IN/OUT)
- new net: R?.1, SW?.2, SW?.2, SW?.2, SW?.2, SW?.2, SW?.2, SW?.2, SW?.2, SW?.5, SW?.5, SW?.5, SW?.5, SW?.5, SW?.5, SW?.5, U?.3 (CH1)
- new net: RV?.2, U?.14 (X1) (x2)
- new net: Q?.2 (E), RV?.E (x8)
- new net: RV?.2, U?.1 (X4) (x2)
- new net: RV?.2, U?.12 (X3) (x2)
- new net: RV?.2, U?.13 (X0) (x2)
- new net: RV?.2, U?.15 (X2) (x2)
- new net: RV?.2, U?.2 (X6) (x2)
- new net: RV?.2, U?.4 (X7) (x2)
- new net: RV?.2, U?.5 (X5) (x2)
- new net: R?.1, R?.2, SW?.1, SW?.6 (x6)
- new net: Q?.1 (B), R?.2 (x8)
- new net: Q?.3 (C), Q?.3 (C), Q?.3 (C), Q?.3 (C), Q?.3 (C), Q?.3 (C), Q?.3 (C), Q?.3 (C), R?.2
- new net: SW?.1, U?.1 (GPB0)
- new net: SW?.1, U?.2 (GPB1)
- new net: SW?.1, U?.21 (GPA0)
- new net: SW?.1, U?.22 (GPA1)
- new net: SW?.3, U?.23 (GPA2)
- new net: SW?.1, U?.24 (GPA3)
- new net: SW?.1, U?.27 (GPA6)
- new net: SW?.1, U?.3 (GPB2)
- new net: SW?.1, U?.5 (GPB4)
- new net: SW?.1, U?.6 (GPB5)
- new net: SW?.1, U?.7 (GPB6)
- new net: SW?.1, U?.8 (GPB7)
- new net: R?.1, R?.2, SW?.1
- new net: U?.12 (+), U?.3 (IN/OUT)
- new net: R?.1, R?.2, U?.1
- new net: R?.1, R?.2, U?.2 (-)
- new net: RV?.2, U?.3 (+)
- new net: R?.1, R?.2, U?.6 (-)
- new net: R?.1, RV?.1, U?.1 (I/O), U?.7
- new net: C?.1, RV?.2, RV?.3, SW?.2 (B), U?.10 (+), U?.8 (O/I)
- new net: R?.2, U?.8, U?.9 (-)
- new net: R?.2, U?.13 (-), U?.14
- new net: R?.2, RV?.1
- new net: R?.2, RV?.3
- new net: R?.1, RV?.1
- new net: R?.2, RV?.2, RV?.3
- new net: C?.1, SW?.3 (C)
- new net: Q?.3 (C), R?.1, U?.6 (OFF)
- new net: Q?.1 (B), R?.1
- new net CHAIN_IN: U?.25 (GPA4)
- new net CHAIN_OUT: U?.26 (GPA5)
- new net CV2_OUT: R?.1
- new net PITCH_CV_OUT: R?.1
- new net PORTEXP_INT: U?.20 (INTA)
- new net SLIDE_OFF: R?.2
- new net SPI_CS_ADC: U?.1 (CS)
- new net SPI_CS_PE: U?.11 (CS)
- new net SPI_MISO: U?.14 (SO), U?.6 (DOUT)
- new net VEE: R?.2, RV?.3, RV?.3, RV?.3, RV?.3, RV?.3, RV?.3, RV?.3, RV?.3, U?.11 (V-), U?.7 (V-), U?.7 (VEE)
- no-connect marks 0 -> 23
Other:
- note added: "Actually TODO put slide circuit before scaling, simpler switching"
- note added: "Amp"
- note added: "Analog Multiplexers"
- note added: "CV2 input potentiometers"
- note added: "Chain input"
- note added: "Chain output"
- note added: "DC offset"
- note added: "Down arrow"
- note added: "Gate mode"
- note added: "Load"
- note added: "Non-panel\nswitch\nfor longer\nslide times"
- note added: "Note:\nThis signal is high to turn slide off.\nWith the curren switch, this makes\nno sense because it's a NC one.\nHowver it'll be replaced with an\nNO open one."
- note added: "Output pitch CV scaling"
- note added: "Output pitch slide"
- note added: "Param select A"
- note added: "Param select B"
- note added: "Pitch CV input voltage (0-5V), to be quantized, scaled"
- note added: "Pitch CV\nInput potentiometers"
- note added: "Reset"
- note added: "Run / stop button - different style"
- note added: "Save"
- note added: "Scale"
- note added: "Sequence mode"
- note added: "Slide"
- note added: "Slide potentiometer LED drivers"
- note added: "Slide time\nPot"
- note added: "Step repeat"
- note added: "Step select voltage"
- note added: "TODO replace with \nTI TS12A4517D (8 pin SOIC)\n"
- note added: "TRIM"
- note added: "Up arrow\n"
- note removed: "3 to 8 decoder\n"
- note removed: "Analog multiplexers\n"
- note removed: "Components to add:\n\n- MCP3202 (ADC)\n- MCP23S17 (Port expander)\n- Slide pots (import from envelope gen)\n- transistors and resistors to drive LEDs\n"
- note removed: "DAC"
- note removed: "TODO verify display pinout\n"
- moved on the sheet: U?

Commit message: Finish Sequencer schematic
Parts:
- removed U?: ATmega32U4-AU, symbol ATmega32U4-AU
- removed U?: DG417, symbol DG417
- added C1, C2: 22p, symbol C
- added C10, C11, C12, C14, C16, C5, C6, C7, C8, C9: 10u, symbol CP
- added C13, C15, C17, C19, C21, C23: 100n, symbol C
- added C20: 1u, symbol CP
- added C3, C4: 470u, symbol CP
- added P1, P3: CONN_01X03, symbol CONN_01X03
- added P2, P4, P5: CONN_02X03, symbol CONN_02X03
- added P6: CONN_01X02, symbol CONN_01X02
- added Q1: MMBT3904, SOT-23, symbol MMBT3904
- added R2: 100R, symbol R
- added R3: 10k, symbol R
- added SW11: LED-BUTTON, symbol LED-BUTTON
- added U11: MC14551B, symbol MC14551B
- added U3: ATmega32U4-AU(edit), symbol ATmega32U4-AU(edit)
- added U9: TS12A4517, symbol TS12A4517
- added X1: CRYSTAL_SMD2, symbol CRYSTAL_SMD2
- gave numbers to parts that had none: 92
Connections:
- net CHAIN_IN: now also P2.5 (P5)
- net CHAIN_OUT: now also P5.5 (P5)
- net CV2_OUT: now also P5.2 (P2), P6.2 (P2)
- net DECODER_ENABLE: now also U3.31 ((OC3A/~OC4A~)PC6)
- net GND: now also C1.2, C10.1, C11.2, C12.2, C13.2, C14.2, C15.2, C16.2, C17.2, C19.2, C2.2, C20.2, C21.2, C23.2, C3.2, C4.1, C5.2, C6.1, C7.2, C8.1, C9.2, P1.2 (P2), P2.6 (P6), P4.6 (P6), P5.6 (P6), SW11.2 (K), SW11.4 (SW2), U11.8 (VSS), U3.15 (GND), U3.23 (GND), U3.35 (GND), U3.43 (GND), X1.2 (GND), X1.4 (GND)
- net PITCH_CV_OUT: now also P5.1 (P1), P6.1 (P1)
- net PORTEXP_INT: now also U3.18 ((OC0B/SCL/INT0)PD0)
- net SLIDE_OFF: now also U3.20 ((RXD/INT2)PD2)
- net SPI_CS_ADC: now also U3.27 ((T0/OC4D/ADC10)PD7)
- net SPI_CS_DAC: now also U3.38 ((ADC5/TMS)PF5)
- net SPI_CS_DISPLAY: now also U3.29 ((ADC12/OC1A/~OC4B~/PCINT12)PB5)
- net SPI_CS_PE: now also U3.36 ((ADC7/TDI)PF7)
- net SPI_MISO: now also P4.1 (P1), U3.11 ((PDO/MISO/PCINT3)PB3)
- net SPI_MOSI: now also P4.4 (P4), U3.10 ((PDI/MOSI/PCINT2)PB2)
- net SPI_SCK: now also P4.3 (P3), U3.9 ((SCLK/PCINT1)PB1)
- net STEP_A0: now also U3.37 ((ADC6/TDO)PF6)
- net STEP_A1: now also U3.39 ((ADC4/TCK)PF4)
- net STEP_A2: now also U3.25 ((ICP2/ADC8)PD4)
- net VCC: now also U8.4 (V+), C11.1, C12.1, C13.1, C14.1, C15.1, C16.1, C17.1, C19.1, C20.1, C21.1, C23.1, C3.1, C5.1, C7.1, C9.1, P1.3 (P3), P4.2 (P2), R2.2, U11.16 (VDD), U3.14 (VCC), U3.2 (UVCC), U3.24 (AVCC), U3.34 (VCC), U3.44 (AVCC), U9.4 (V+); no longer U8.4 (V+)
- net VEE: now also C10.2, C4.2, C6.2, C8.2, P1.1 (P1), U11.7 (VEE), U9.7 (V-)
- net at R30.1, SW13.2, SW13.5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: now also SW17.5
- net at U2.4 (GPB3): now also SW11.1 (SW1)
- net at R19.1, R23.2, SW17.1: now also SW17.6
- net at U8.12 (+): now also U11.4 (X); no longer U7.3 (IN/OUT)
- net at R20.1, RV13.1, U8.7: now also U9.1 (COM)
- net PITCH_CV: now reaches C18.1, RV13.2, RV13.3, SW19.2 (B)
- net PITCH_CV: now also U11.15 (W0), U9.8 (NC); no longer U8.10 (+)
- net at Q3.3 (C), R14.1: now also U9.6 (IN)
- new net: Q1.2 (E), SW11.3 (A)
- new net: Q1.1 (B), R3.2
- new net: Q1.3 (C), R2.1
- new net: C1.1, U3.17 (XTAL1), X1.1
- new net: C2.1, U3.16 (XTAL2), X1.3
- new net: U11.14 (W), U8.10 (+)
- new net CHAIN_CV2: P2.2 (P2), U11.3 (X1)
- new net CHAIN_GATE: P2.3 (P3), U11.10 (Y1)
- new net CHAIN_PITCH_CV: P2.1 (P1), U11.1 (W1)
- new net CHAIN_TRIGGER: P2.4 (P4), U11.12 (Z1)
- new net CV2: U11.2 (X0), U7.3 (IN/OUT)
- new net EXTERNAL_CLOCK: P3.1 (P1), U3.1 ((INT6/AIN0)PE6)
- new net GATE: U11.6 (Y0), U3.30 ((ADC13/OC1B/OC4B/PCINT13)PB6)
- new net GATE_OUT: P3.2 (P2), P5.3 (P3), U11.5 (Y)
- new net ISP_RESET: P4.5 (P5), U3.13 (RESET)
- new net ROUTE_CHAINED: U11.9 (CONTROL), U3.21 ((TXD/INT3)PD3)
- new net RUN_INDICATOR: R3.1, U3.28 ((ADC11/PCINT4)PB4)
- new net TRIGGER: U11.11 (Z0), U3.19 ((SDA/INT1)PD1)
- new net TRIGGER_OUT: P3.3 (P3), P5.4 (P4), U11.13 (Z)
- no-connect marks 23 -> 37
Other:
- note added: "+5V"
- note added: "-5V"
- note added: "0, RX"
- note added: "0V"
- note added: "1, TX"
- note added: "18, A0"
- note added: "19, A1"
- note added: "2, SDA"
- note added: "20, A2"
- note added: "21, A3"
- note added: "3, SCL"
- note added: "4, A6"
- note added: "5"
- note added: "6, A7"
- note added: "7"
- note added: "ADC"
- note added: "Board\ndecoupling"
- note added: "CV Buffers"
- note added: "Chain input\nconnector"
- note added: "Chain output\nconnector"
- note added: "Chain\nMux"
- note added: "DAC"
- note added: "Decoder"
- note added: "Decoupling capacitors"
- note added: "Disp\nDriver"
- note added: "Display + additional indication LEDs"
- note added: "IO10, A10"
- note added: "IO8, A8"
- note added: "IO9, A9"
- note added: "ISP Connector"
- note added: "MISO, 14"
- note added: "MOSI, 16"
- note added: "Microcontroller"
- note added: "Mux"
- note added: "Opamp"
- note added: "Output Pitch CV DAC"
- note added: "POWER"
- note added: "Port expander for digital I/O\n(mainly buttons)"
- note added: "Portexp"
- note added: "Run / stop"
- note added: "SCK, 15"
- note added: "Switch between outputting\nlocal signals, or chained in signals"
- note added: "To banana connectors"
- note added: "uC"
- note removed: "Actually TODO put slide circuit before scaling, simpler switching"
- note removed: "Note:\nThis signal is high to turn slide off.\nWith the curren switch, this makes\nno sense because it's a NC one.\nHowver it'll be replaced with an\nNO open one."
- note removed: "Run / stop button - different style"
- note removed: "TODO replace with \nTI TS12A4517D (8 pin SOIC)\n"
- moved on the sheet: AFF1, C18, C22, D1, D2, D3, Q10, Q2, Q3, Q4, Q5, Q6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

Commit message: Most of sequencer PCB design + aligning stuff with panel
Still need to route power connections
Parts:
- AFF1: footprint (none) -> CC04-41SURKWA:CC04-41SURKWA
- C1, C18, C2: footprint (none) -> Capacitors_SMD:C_0603
- C10, C11, C12, C14, C16, C20, C22, C5, C6, C7, C8, C9: footprint (none) -> Capacitors_SMD:C_0805
- C13, C15, C17, C19, C21, C23: footprint (none) -> Capacitors_SMD:C_0402
- C3, C4: footprint (none) -> Capacitors_ThroughHole:CP_Radial_D8.0mm_P3.50mm
- D1, D2, D3: footprint (none) -> LEDs:LED_D3.0mm
- P1, P3: footprint (none) -> Connectors_Molex:Molex_KK-6410-03_03x2.54mm_Straight
- P2, P4, P5: footprint (none) -> Pin_Headers:Pin_Header_Straight_2x03_Pitch2.54mm
- P6: footprint (none) -> Connectors_Molex:Molex_KK-6410-02_02x2.54mm_Straight
- Q1, Q10, Q2, Q3, Q4, Q5, Q6, Q7, Q8, Q9: footprint SOT-23 -> TO_SOT_Packages_SMD:SOT-23
- R1, R17, R2, R31, R32, R7, R9: footprint (none) -> Resistors_SMD:R_1206
- R10, R11, R12, R14, R15, R16, R18, R20, R21, R22, R24, R26, R27, R29, R3, R6: footprint (none) -> Resistors_SMD:R_0603
- R13, R19, R23, R25, R28, R30, R4, R5, R8: footprint (none) -> Resistors_SMD:R_0805
- RV1, RV10: footprint (none) -> Potentiometers:Potentiometer_Triwood_RM-065
- RV11, RV13, RV14, RV15, RV2, RV4, RV5, RV7, RV8: footprint (none) -> Potentiometers:Potentiometer_Bourns_PTV09A-1_Horizontal
- RV12, RV16, RV17, RV18, RV19, RV3, RV6, RV9: footprint (none) -> Bourns PTL:Bourns-PTL30-X
- SW1, SW10, SW2, SW3, SW4, SW5, SW6, SW7, SW8, SW9: footprint (none) -> Buttons_Switches_ThroughHole:SW_PUSH_6mm
- SW11: footprint (none) -> 5GTH9:5GTH9
- SW12: footprint (none) -> MHS123K:MHS123K
- SW13, SW14, SW15, SW16, SW17, SW18, SW20, SW21: footprint (none) -> 6-pin-momentary-push-button:6-pin-momentary-push-button
- SW19: footprint (none) -> Pin_Headers:Pin_Header_Straight_1x03_Pitch2.54mm
- U1: footprint (none) -> SMD_Packages:SOIC-24
- U10, U4, U9: footprint (none) -> SMD_Packages:SOIC-8-N
- U11, U5, U6, U7: footprint (none) -> SMD_Packages:SO-16-N
- U2: footprint (none) -> SMD_Packages:SOIC-28
- U3: footprint (none) -> Housings_QFP:TQFP-44_10x10mm_Pitch0.8mm
- U8: footprint (none) -> SMD_Packages:SOIC-14_N
- X1: footprint (none) -> Crystals:Crystal_SMD_3225-4pin_3.2x2.5mm
Connections:
- net PITCH_CV: now also RV13.1; no longer RV13.3
- net at R20.1, U8.7, U9.1 (COM): now also RV13.3; no longer RV13.1

Commit message: Add screw holes to seq. PCB, finish panel alignment
Parts:
- added C24, C25: 10u, Capacitors_SMD:C_0805, symbol CP
Connections:
- net GND: now also C24.2, C25.1
- net VCC: now also C24.1
- net VEE: now also C25.2
Other:
- note added: "Slide\nSw"
Changed lines of the file:
@@
 $EndComp
 Wire Wire Line
-	6750 9950 10750 9950
+	6750 9950 11050 9950
 $Comp
 L CP C3
@@
 	6800 9500 6800 9850
 Wire Wire Line
-	6750 9550 10750 9550
+	6750 9550 11050 9550
 Wire Wire Line
 	7200 9550 7200 9600
@@
 	6800 10050 6800 10400
 Wire Wire Line
-	6750 10350 8000 10350
+	6750 10350 11050 10350
 Wire Wire Line
 	7200 10350 7200 10300
@@
 Wire Wire Line
 	9500 7300 9500 7150
+$Comp
+L CP C24
+U 1 1 5A883D7F
+P 11050 9750
+F 0 "C24" H 11075 9850 50  0000 L CNN
+F 1 "10u" H 11075 9650 50  0000 L CNN
+F 2 "Capacitors_SMD:C_0805" H 11088 9600 50  0001 C CNN
+F 3 "" H 11050 9750 50  0000 C CNN
+	1    11050 9750
+	1    0    0    -1
+$EndComp
+$Comp
+L CP C25
+U 1 1 5A8840DB
+P 11050 10150
+F 0 "C25" H 11075 10250 50  0000 L CNN
+F 1 "10u" H 11075 10050 50  0000 L CNN
+F 2 "Capacitors_SMD:C_0805" H 11088 10000 50  0001 C CNN
+F 3 "" H 11050 10150 50  0000 C CNN
+	1    11050 10150
+	1    0    0    -1
+$EndComp
+Wire Wire Line
+	11050 9550 11050 9600
+Connection ~ 10750 9550
+Wire Wire Line
+	11050 9900 11050 10000
+Connection ~ 11050 9950
+Connection ~ 10750 9950
+Wire Wire Line
+	11050 10350 11050 10300
+Connection ~ 8000 10350
+Text Notes 11100 10500 2    40   ~ 0
+Slide\nSw
 $EndSCHEMATC

Commit message: Add test points, finish silkscreen on sequencer board
Parts:
- added W?: PITCH_CV, symbol TEST_1P
- added W?: STEP_SELECT, symbol TEST_1P
- added W?: CV2, symbol TEST_1P
- R13, R19, R23, R25, R28, R4, R5, R8: value 1k -> 1k, .1%
Connections:
- wire segments 620 -> 622
Changed lines of the file:
@@
 U 1 1 5A75E9F2
 P 6500 5650
-F 0 "R5" V 6400 5650 50  0000 C CNN
-F 1 "1k" V 6500 5650 50  0000 C CNN
+F 0 "R5" V 6350 5650 50  0000 C CNN
+F 1 "1k, .1%" V 6400 5650 50  0000 C CNN
 F 2 "Resistors_SMD:R_0805" V 6430 5650 50  0001 C CNN
 F 3 "" H 6500 5650 50  0000 C CNN
@@
 U 1 1 5A760D7E
 P 7350 5650
-F 0 "R8" V 7250 5650 50  0000 C CNN
-F 1 "1k" V 7350 5650 50  0000 C CNN
+F 0 "R8" V 7200 5650 50  0000 C CNN
+F 1 "1k, .1%" V 7250 5650 50  0000 C CNN
 F 2 "Resistors_SMD:R_0805" V 7280 5650 50  0001 C CNN
 F 3 "" H 7350 5650 50  0000 C CNN
@@
 U 1 1 5A764493
 P 8200 5650
-F 0 "R13" V 8100 5650 50  0000 C CNN
-F 1 "1k" V 8200 5650 50  0000 C CNN
+F 0 "R13" V 8050 5650 50  0000 C CNN
+F 1 "1k, .1%" V 8100 5650 50  0000 C CNN
 F 2 "Resistors_SMD:R_0805" V 8130 5650 50  0001 C CNN
 F 3 "" H 8200 5650 50  0000 C CNN
@@
 U 1 1 5A7644A7
 P 9050 5650
-F 0 "R19" V 8950 5650 50  0000 C CNN
-F 1 "1k" V 9050 5650 50  0000 C CNN
+F 0 "R19" V 8900 5650 50  0000 C CNN
+F 1 "1k, .1%" V 8950 5650 50  0000 C CNN
 F 2 "Resistors_SMD:R_0805" V 8980 5650 50  0001 C CNN
 F 3 "" H 9050 5650 50  0000 C CNN
@@
 U 1 1 5A765425
 P 9900 5650
-F 0 "R23" V 9800 5650 50  0000 C CNN
-F 1 "1k" V 9900 5650 50  0000 C CNN
+F 0 "R23" V 9750 5650 50  0000 C CNN
+F 1 "1k, .1%" V 9800 5650 50  0000 C CNN
 F 2 "Resistors_SMD:R_0805" V 9830 5650 50  0001 C CNN
 F 3 "" H 9900 5650 50  0000 C CNN
@@
 U 1 1 5A765439
 P 10750 5650
-F 0 "R25" V 10650 5650 50  0000 C CNN
-F 1 "1k" V 10750 5650 50  0000 C CNN
+F 0 "R25" V 10600 5650 50  0000 C CNN
+F 1 "1k, .1%" V 10650 5650 50  0000 C CNN
 F 2 "Resistors_SMD:R_0805" V 10680 5650 50  0001 C CNN
 F 3 "" H 10750 5650 50  0000 C CNN
@@
 U 1 1 5A765453
 P 11600 5650
-F 0 "R28" V 11500 5650 50  0000 C CNN
-F 1 "1k" V 11600 5650 50  0000 C CNN
+F 0 "R28" V 11450 5650 50  0000 C CNN
+F 1 "1k, .1%" V 11500 5650 50  0000 C CNN
 F 2 "Resistors_SMD:R_0805" V 11530 5650 50  0001 C CNN
 F 3 "" H 11600 5650 50  0000 C CNN
@@
 U 1 1 5A770C73
 P 5600 5650
-F 0 "R4" V 5500 5650 50  0000 C CNN
-F 1 "1k" V 5600 5650 50  0000 C CNN
+F 0 "R4" V 5450 5650 50  0000 C CNN
+F 1 "1k, .1%" V 5500 5650 50  0000 C CNN
 F 2 "Resistors_SMD:R_0805" V 5530 5650 50  0001 C CNN
 F 3 "" H 5600 5650 50  0000 C CNN
@@
 	6000 4650 5800 4650
 Wire Wire Line
-	5800 4650 5800 4900
+	5800 4650 5800 5000
 Wire Wire Line
 	5950 4900 5950 4850
@@
 	11700 3950 11750 3950
 Wire Wire Line
-	12400 5350 12400 6400
+	12400 6400 12400 5300
 Connection ~ 5950 1050
 Wire Wire Line
@@
 Text GLabel 10900 7150 2    40   Output ~ 0
 PITCH_CV
-Text GLabel 5800 4900 3    40   Output ~ 0
+Text GLabel 5800 5000 3    40   Output ~ 0
 CV2
 Wire Wire Line
@@
 Text Notes 11100 10500 2    40   ~ 0
 Slide\nSw
+$Comp
+L TEST_1P W?
+U 1 1 5A8BFD05
+P 10750 7100
+F 0 "W?" H 10750 7370 50  0000 C CNN
+F 1 "PITCH_CV" H 10750 7300 50  0000 C CNN
+F 2 "" H 10950 7100 50  0000 C CNN
+F 3 "" H 10950 7100 50  0000 C CNN
+	1    10750 7100
+	1    0    0    -1
+$EndComp
+Wire Wire Line
+	10750 7100 10750 7150
+Connection ~ 10750 7150
+$Comp
+L TEST_1P W?
+U 1 1 5A8C6D75
+P 12400 5300
+F 0 "W?" H 12400 5570 50  0000 C CNN
+F 1 "STEP_SELECT" H 12400 5500 50  0000 C CNN
+F 2 "" H 12600 5300 50  0000 C CNN
+F 3 "" H 12600 5300 50  0000 C CNN
+	1    12400 5300
+	1    0    0    -1
+$EndComp
+Connection ~ 12400 5350
+$Comp
+L TEST_1P W?
+U 1 1 5A8CD1D0
+P 5750 4900
+F 0 "W?" H 5750 5170 50  0000 C CNN
+F 1 "CV2" H 5750 5100 50  0000 C CNN
+F 2 "" H 5950 4900 50  0000 C CNN
+F 3 "" H 5950 4900 50  0000 C CNN
+	1    5750 4900
+	0    -1   -1   0
+$EndComp
+Wire Wire Line
+	5750 4900 5800 4900
+Connection ~ 5800 4900
 $EndSCHEMATC

Commit message: Finish sequencer PCB (and sent off for fab at this point)
Parts:
- W1, W2, W3: renamed from W?; footprint (none) -> Measurement_Points:Measurement_Point_Round-SMD-Pad_Big
Changed lines of the file:
@@
 Slide\nSw
 $Comp
-L TEST_1P W?
+L TEST_1P W2
 U 1 1 5A8BFD05
 P 10750 7100
-F 0 "W?" H 10750 7370 50  0000 C CNN
+F 0 "W2" H 10750 7370 50  0000 C CNN
 F 1 "PITCH_CV" H 10750 7300 50  0000 C CNN
-F 2 "" H 10950 7100 50  0000 C CNN
+F 2 "Measurement_Points:Measurement_Point_Round-SMD-Pad_Big" H 10950 7100 50  0001 C CNN
 F 3 "" H 10950 7100 50  0000 C CNN
 	1    10750 7100
@@
 Connection ~ 10750 7150
 $Comp
-L TEST_1P W?
+L TEST_1P W3
 U 1 1 5A8C6D75
 P 12400 5300
-F 0 "W?" H 12400 5570 50  0000 C CNN
+F 0 "W3" H 12400 5570 50  0000 C CNN
 F 1 "STEP_SELECT" H 12400 5500 50  0000 C CNN
-F 2 "" H 12600 5300 50  0000 C CNN
+F 2 "Measurement_Points:Measurement_Point_Round-SMD-Pad_Big" H 12600 5300 50  0001 C CNN
 F 3 "" H 12600 5300 50  0000 C CNN
 	1    12400 5300
@@
 Connection ~ 12400 5350
 $Comp
-L TEST_1P W?
+L TEST_1P W1
 U 1 1 5A8CD1D0
 P 5750 4900
-F 0 "W?" H 5750 5170 50  0000 C CNN
+F 0 "W1" H 5750 5170 50  0000 C CNN
 F 1 "CV2" H 5750 5100 50  0000 C CNN
-F 2 "" H 5950 4900 50  0000 C CNN
+F 2 "Measurement_Points:Measurement_Point_Round-SMD-Pad_Big" H 5950 4900 50  0001 C CNN
 F 3 "" H 5950 4900 50  0000 C CNN
 	1    5750 4900
